Commit message: sensore di prossimità inserito

File: urdf/my_robot_x.urdf (robot description, URDF)
Before this commit: robot my_robot, 5 links, 4 joints
Links:
- added link hokuyo_link; visual box size=0.05 0.05 0.05
Joints:
- added joint hokuyo_joint: type fixed, parent base_link, child hokuyo_link, origin xyz=0.125 0 0.0325 rpy=0 0 0

File: urdf/my_robot_x.xacro (robot description, xacro)
@@ -3,4 +3,5 @@
   <xacro:include filename="$(find my_robot_urdf)/urdf/cylinder_wheel.urdf.xacro"/>
   <xacro:include filename="$(find my_robot_urdf)/urdf/caster_wheel.urdf.xacro"/>
+  <xacro:include filename="$(find my_robot_urdf)/urdf/visual_sensor.xacro"/>
   <link name="base_link">
     <visual>
@@ -21,4 +22,5 @@
   <cylinder_wheel fb="front" lr="right" parent="base_link" translateX="0" translateY="0.5" flipY="1"/>
   <cylinder_wheel fb="front" lr="left" parent="base_link" translateX="0" translateY="-0.5" flipY="1"/>
+  <hokuyo base_radius="${base_radius}" base_height="${base_height}"/>
   <gazebo>
     <plugin name="gazebo_ros_control" filename="libgazebo_ros_control.so">
